File: Boards/Round 2 PCB/PCB_R2.kicad_sch (KiCad schematic)
At the start: 67 parts, among them J1 Screw_Terminal_01x12, J10 Screw_Terminal_01x03, J11 Screw_Terminal_01x12, J12 Screw_Terminal_01x03, J13 Screw_Terminal_01x03, J14 Screw_Terminal_01x03, J15 Screw_Terminal_01x03, J16 Screw_Terminal_01x03, J17 Screw_Terminal_01x03, J18 Screw_Terminal_01x03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

Commit message: ground layer test
placed all transistors, about to delete all ground connections
Parts:
- added Q1, Q10, Q11, Q12, Q2, Q3, Q4, Q5, Q6, Q7, Q8, Q9: NMOS, Package_TO_SOT_SMD:SOT-23-3, symbol Simulation_SPICE:NMOS
Connections:
- net +3.3V: now also Q1.1 (D), Q10.1 (D), Q11.1 (D), Q12.1 (D), Q2.1 (D), Q3.1 (D), Q4.1 (D), Q5.1 (D), Q6.1 (D), Q7.1 (D), Q8.1 (D), Q9.1 (D)
- net M0: now also Q1.3 (S); no longer U1.14 (PA0)
- net M1: now also Q2.3 (S); no longer U1.15 (PA1)
- net M10: now also Q11.3 (S); no longer U1.43 (PA10)
- net M11: now also Q12.3 (S); no longer U1.40 (PC9)
- net M2: now also Q3.3 (S); no longer U1.16 (PA2)
- net M3: now also Q4.3 (S); no longer U1.17 (PA3)
- net M4: now also Q5.3 (S); no longer U1.20 (PA4)
- net M5: now also Q6.3 (S); no longer U1.21 (PA5)
- net M6: now also Q7.3 (S); no longer U1.22 (PA6)
- net M7: now also Q8.3 (S); no longer U1.23 (PA7)
- net M8: now also Q9.3 (S); no longer U1.41 (PA8)
- net M9: now also Q10.3 (S); no longer U1.42 (PA9)
- new net T0: Q1.2 (G), U1.14 (PA0)
- new net T1: Q2.2 (G), U1.15 (PA1)
- new net T10: Q11.2 (G), U1.43 (PA10)
- new net T11: Q12.2 (G), U1.40 (PC9)
- new net T2: Q3.2 (G), U1.16 (PA2)
- new net T3: Q4.2 (G), U1.17 (PA3)
- new net T4: Q5.2 (G), U1.20 (PA4)
- new net T5: Q6.2 (G), U1.21 (PA5)
- new net T6: Q7.2 (G), U1.22 (PA6)
- new net T7: Q8.2 (G), U1.23 (PA7)
- new net T8: Q9.2 (G), U1.41 (PA8)
- new net T9: Q10.2 (G), U1.42 (PA9)
Other:
- moved on the sheet: D3, J20, J21, J9, JP1, R12, R17, R18, R19

Commit message: HVPS Update
changed HVPS components to increase maximum current from 0.5A to 1A
Parts:
- C14, C15: value 180uF -> 47uF
- C8, C9: value 20nF -> 10nF
- L1: value 60uH -> 0.27uH
- L2: value 2.2uH -> 0.33uH
Changed lines of the file:
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@@
       (effects (font (size 1.27 1.27)))
     )
-    (property "Value" "2.2uH" (at 100.33 172.72 90)
+    (property "Value" "0.33uH" (at 100.33 172.72 90)
       (effects (font (size 1.27 1.27)))
     )
@@
       (effects (font (size 1.27 1.27)) hide)
     )
-    (property "Datasheet" "~" (at 100.33 175.26 0)
+    (property "Datasheet" "or 10uH" (at 100.33 175.26 0)
       (effects (font (size 1.27 1.27)) hide)
     )
@@
       (effects (font (size 1.27 1.27)) (justify left))
     )
-    (property "Value" "20nF" (at 81.28 152.4 0)
+    (property "Value" "10nF" (at 81.28 152.4 0)
       (effects (font (size 1.27 1.27)) (justify left))
     )
@@
       (effects (font (size 1.27 1.27)) (justify left))
     )
-    (property "Value" "180uF" (at 124.46 157.48 0)
+    (property "Value" "47uF" (at 124.46 157.48 0)
       (effects (font (size 1.27 1.27)) (justify left))
     )
@@
       (effects (font (size 1.27 1.27)) (justify left))
     )
-    (property "Value" "180uF" (at 124.46 185.42 0)
+    (property "Value" "47uF" (at 124.46 185.42 0)
       (effects (font (size 1.27 1.27)) (justify left))
     )
@@
       (effects (font (size 1.27 1.27)))
     )
-    (property "Value" "60uH" (at 100.33 144.78 90)
+    (property "Value" "0.27uH" (at 100.33 144.78 90)
       (effects (font (size 1.27 1.27)))
     )
@@
       (effects (font (size 1.27 1.27)) hide)
     )
-    (property "Datasheet" "~" (at 100.33 147.32 0)
+    (property "Datasheet" "or 12uH" (at 100.33 147.32 0)
       (effects (font (size 1.27 1.27)) hide)
     )
@@
       (effects (font (size 1.27 1.27)) (justify left))
     )
-    (property "Value" "20nF" (at 81.28 180.34 0)
-      (effects (font (size 1.27 1.27)) (justify left))
-    )
+    (property "Value" "10nF" (at 81.28 180.34 0)
+      (effects (font (size 1.27 1.27)) (justify left))
+    )
